File: Hardware/0_8mm_Layers.sch (EAGLE design)
At the start: 59 parts, among them J1 AVR_SPI_PROG_3X2TESTPOINTS, Q1 220mA/50V/3.5Ω, Q2 220mA/50V/3.5Ω, Q3 220mA/50V/3.5Ω, U1 ATTINY861V-10MU

Commit message: Board and Code changes. Close to v1.0
Board and Code changes. Close to v1.0
Connections:
- removed net 14: U1.PB6(14/A9/INT0)
- net GND: now also J10.1
- net IR_DETECTOR: now also U1.PB6(14/A9/INT0)
- net N$45: now also D1.A; no longer D1.C
- net N$46: now also D1.C; no longer D1.A
- net V_BATT: now also J9.1
Other:
- moved on the sheet: D1
Changed lines of the file:
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@@
 <part name="R1" library="SparkFun-Resistors" deviceset="1KOHM" device="-0603-1/10W-1%" value="1k"/>
 <part name="D1" library="SparkFun-LED" deviceset="LED-IR" device="0603" value="IR LED"/>
+<part name="GND11" library="SparkFun-PowerSymbols" deviceset="GND" device=""/>
 </parts>
 <sheets>
@@
 <attribute name="VALUE" x="223.52" y="49.784" size="1.778" layer="96" font="vector" rot="R180" align="top-center"/>
 </instance>
-<instance part="D1" gate="G$1" x="220.98" y="40.64" smashed="yes" rot="R90">
-<attribute name="NAME" x="225.552" y="37.211" size="1.778" layer="95" font="vector" rot="R180"/>
-<attribute name="VALUE" x="225.552" y="42.545" size="1.778" layer="96" font="vector" rot="R180" align="top-left"/>
+<instance part="D1" gate="G$1" x="223.52" y="40.64" smashed="yes" rot="R270">
+<attribute name="NAME" x="218.948" y="44.069" size="1.778" layer="95" font="vector"/>
+<attribute name="VALUE" x="218.948" y="38.735" size="1.778" layer="96" font="vector" align="top-left"/>
+</instance>
+<instance part="GND11" gate="1" x="48.26" y="147.32" smashed="yes">
+<attribute name="VALUE" x="48.26" y="147.066" size="1.778" layer="96" align="top-center"/>
 </instance>
 </instances>
@@
 <pinref part="GND3" gate="1" pin="GND"/>
 </segment>
+<segment>
+<pinref part="J10" gate="G$1" pin="1"/>
+<wire x1="45.72" y1="152.4" x2="48.26" y2="152.4" width="0.1524" layer="91"/>
+<wire x1="48.26" y1="152.4" x2="48.26" y2="149.86" width="0.1524" layer="91"/>
+<pinref part="GND11" gate="1" pin="GND"/>
+</segment>
 </net>
 <net name="N$6" class="0">
@@
 <wire x1="81.28" y1="53.34" x2="81.28" y2="55.88" width="0.1524" layer="91"/>
 <pinref part="SUPPLY5" gate="G$1" pin="V_BATT"/>
+</segment>
+<segment>
+<pinref part="J9" gate="G$1" pin="1"/>
+<wire x1="45.72" y1="160.02" x2="48.26" y2="160.02" width="0.1524" layer="91"/>
+<label x="48.26" y="160.02" size="1.27" layer="95" xref="yes"/>
 </segment>
 </net>
@@
 <label x="226.06" y="81.28" size="1.27" layer="95" xref="yes"/>
 </segment>
+<segment>
+<pinref part="U1" gate="A" pin="PB6(14/A9/INT0)"/>
+<wire x1="68.58" y1="43.18" x2="71.12" y2="43.18" width="0.1524" layer="91"/>
+<label x="71.12" y="43.18" size="1.27" layer="95" xref="yes"/>
+</segment>
 </net>
 <net name="!RESET" class="0">
@@
 </segment>
 </net>
-<net name="14" class="0">
-<segment>
-<pinref part="U1" gate="A" pin="PB6(14/A9/INT0)"/>
-<wire x1="68.58" y1="43.18" x2="71.12" y2="43.18" width="0.1524" layer="91"/>
-<label x="71.12" y="43.18" size="1.27" layer="95" xref="yes"/>
-</segment>
-</net>
 <net name="N$44" class="0">
 <segment>
@@
 <wire x1="228.6" y1="48.26" x2="231.14" y2="48.26" width="0.1524" layer="91"/>
 <wire x1="231.14" y1="48.26" x2="231.14" y2="40.64" width="0.1524" layer="91"/>
-<pinref part="D1" gate="G$1" pin="C"/>
-<wire x1="231.14" y1="40.64" x2="226.06" y2="40.64" width="0.1524" layer="91"/>
+<pinref part="D1" gate="G$1" pin="A"/>
+<wire x1="226.06" y1="40.64" x2="231.14" y2="40.64" width="0.1524" layer="91"/>
 </segment>
 </net>
 <net name="N$46" class="0">
 <segment>
-<pinref part="D1" gate="G$1" pin="A"/>
-<wire x1="218.44" y1="40.64" x2="215.9" y2="40.64" width="0.1524" layer="91"/>
 <wire x1="215.9" y1="40.64" x2="215.9" y2="43.18" width="0.1524" layer="91"/>
 <pinref part="J12" gate="G$1" pin="1"/>
 <wire x1="215.9" y1="43.18" x2="213.36" y2="43.18" width="0.1524" layer="91"/>
-</segment>
-</net>
+<pinref part="D1" gate="G$1" pin="C"/>
+<wire x1="215.9" y1="40.64" x2="218.44" y2="40.64" width="0.1524" layer="91"/>
+</segment>
+</net>
