File: Hardware/Production/CircuitPanel.brd (EAGLE design)
At the start: 116.8 x 86.4 mm, 76 parts, among them J1 AVR_SPI_PROG_3X2TESTPOINTS, Q1 220mA/50V/3.5Ω, Q2 220mA/50V/3.5Ω, Q3 220mA/50V/3.5Ω, U1 ATTINY861V-10MU

Commit message: v10
Parts:
- added BT2: (no value), SparkFun-Batteries:BATTCON_20MM_4LEGS_OVERPASTE_INNER
- added C3, C4, C5, C6: 0.1uF, SparkFun-Capacitors:0603
- added D1S10, D1S11, D1S12, D1S3, D1S8, D1S9, D2S10, D2S11, D2S12, D2S13, D2S14, D2S8, D2S9, D3S10, D3S11, D3S12, D3S13, D3S14, D3S8, D3S9, DIS1: (no value), SparkFun-LED:LED-0603
- added D2, D4, D6: IR PHOTOTRANS, SparkFun-LED:LED-0603
- added D3, D5, D7: IR LED, SparkFun-LED:LED-0603
- added J13: AVR_SPI_PROG_3X2TESTPOINTS, SparkFun-Connectors:2X3_TEST_POINTS
- added J14, J24: (no value), SparkFun-Connectors:1X02
- added J15, J16, J17, J18, J19, J20, J21, J22, J23: (no value), SparkFun-Connectors:1X01
- added Q4, Q5, Q6: 220mA/50V/3.5Ω, SparkFun-DiscreteSemi:SOT23-3
- added R14, R15, R23, R24, R25, R26, R27, R28, R29, R30: 1k, SparkFun-Resistors:0603
- added R16, R17, R18, R19, R20, R21, R22: 33, SparkFun-Resistors:0603
- added S4, S5: MOMENTARY-SWITCH-SPST-SMD-5.2MM-TALL, SparkFun-Switches:TACTILE_SWITCH_SMD_5.2MM
- added S6: (no value), SparkFun-Switches:SWITCH_SPST_SMD_A
- added U$18, U$35: (no value), output:#GITHUB#COM#NPOOLE#BEANCOUNTER#0
- added U$19, U$36: (no value), SparkFun-Aesthetics:OSHW-LOGO-M
- added U$20, U$38: (no value), output:40
- added U$21, U$39: (no value), output:120
- added U$22, U$40: (no value), output:160
- added U$23, U$41: (no value), output:#ON#0
- added U$24, U$42: (no value), output:#OFF#EXT#0
- added U$25, U$43: (no value), output:NPOOLE_20210
- added U$26, U$44: (no value), output:PRESS_THE_COUNT#RESET_BUTTON_TO_CHANGE_THE_PITCH_SETTING0
- added U$27: (no value), output:#RESET_COUNTER#0
- added U$28: (no value), output:#CHANGE_COMPONENT_PITCH#0
- added U$29: (no value), output:QUICK#PRESS_THE_COUNT#RESET_BUTTON_TO_STOP_COUNTING0
- added U$30: (no value), output:QUICK#PRESS_AGAIN_TO_RESUME0
- added U$31: (no value), output:PRESS_AND_HOLD_THE_COUNT#RESET_BUTTON_UNTIL_THE0
- added U$32: (no value), output:DISPLAY_BEGINS_BLINKING_THEN_RELEASE_TO_CLEAR_THE_CURRENT_COUNT0
- added U$33: (no value), output:QUICK#PRESS_THE_SETUP_BUTTON_TO_DISPLAY_THE_COMPONENT_PITCH_IN_MM0
- added U$34: (no value), output:PRESS_THE_SETUP_AGAIN_TO_EXIT_THE_PITCH_MENU0
- added U$37: (no value), output:00
- added U2: ATTINY861V-10MU, Melodica:32M1-A_ATM
- U$1: device output:#COUNT#0 -> logo:LOGO#SVG0
- U$16: device output:PRESS_THE_COUNT#RESET_BUTTON_TO_CHANGE_THE_PITCH_STTING0 -> output:#PAUSE#CONTINUE_COUNTING#0
- U$2: device output:#RESET#0 -> output:#_3V#0
- U$3: device output:#SETUP#0 -> output:#_GND#0
- U$5: device tape:TAPE0603#SVG0 -> output:00
- moved U$5 127.3 mm to (4.84, 3.00)
- moved S1 106.7 mm to (111.8, 16.5), flipped to the top
- moved S2 106.7 mm to (111.8, 3.81), flipped to the top
- moved U$3 104.2 mm to (106.9, 67.1), turned to 180 degrees
- moved U$1 101.1 mm to (108.0, 33.5)
- moved U$2 99.4 mm to (106.9, 56.9), turned to 180 degrees
- moved U$6 97.0 mm to (9.91, 15.2), flipped to the bottom
- moved U$7 97.0 mm to (9.91, 5.08), flipped to the bottom
- moved J10 96.5 mm to (10.2, 5.08), flipped to the top
- moved J7 96.5 mm to (10.2, 0.00), flipped to the top
- moved J8 96.5 mm to (10.2, 20.3), flipped to the top
- moved J9 96.5 mm to (10.2, 15.2), flipped to the top
- moved BT1 90.7 mm to (103.8, 10.4), flipped to the bottom
- moved D23 76.4 mm to (20.2, 5.02), flipped to the top
- moved D3S3 76.2 mm to (96.5, 15.2), flipped to the top
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Connections:
- net IR_DETECTOR renamed IR_DETECTOR_A
- removed net N$6: BT1.1, S3.2
- new net !RESET1: J13.5, R27.1, U2.11
- new net 10: R19.1, U2.22
- new net 10/SCK1: J13.3, R25.1, U2.32
- new net 14: R20.1, U2.17
- new net 15: R21.1, U2.15
- new net 16: R22.1, U2.14
- new net 17: J14.2, U2.2
- new net 18: S4.1, U2.7
- new net 19: S5.1, U2.8
- new net 8: R17.1, U2.25
- new net 8/COPI1: J13.4, R23.1, U2.30
- new net 9: R18.1, U2.23
- new net 9/CIPO1: J13.1, R24.1, U2.31
- new net GND1: BT2.2, C4.2, C5.2, C6.2, J13.6, J14.1, J22.1, Q4.2, Q5.2, Q6.2, R26.1, R29.1, S4.3, S5.3, U2.21, U2.5
- new net IR_DETECTOR_A1: C4.1, D4.C, R26.2, U2.10
- new net IR_DETECTOR_B: C3.1, D2.C, R14.2, U1.13
- new net IR_DETECTOR_B1: C6.1, D6.C, R29.2, U2.13
- new net N$1: BT1.1, S3.3
- new net N$19: Q4.1, R23.2
- new net N$20: D1S10.C, D1S11.C, D1S12.C, D1S3.C, D1S8.C, D1S9.C, DIS1.C, Q4.3
- new net N$21: D2S10.C, D2S11.C, D2S12.C, D2S13.C, D2S14.C, D2S8.C, D2S9.C, Q5.3
- new net N$22: D3S10.C, D3S11.C, D3S12.C, D3S13.C, D3S14.C, D3S8.C, D3S9.C, Q6.3
- new net N$23: Q5.1, R24.2
- new net N$24: Q6.1, R25.2
- new net N$30: BT2.1, S6.3
- new net N$51: D1.A, D3.A, J12.1
- new net N$63: J24.2, R28.1, R30.1
- new net N$64: D5.C, R28.2
- new net N$65: D7.C, R30.2
- new net N$66: D5.A, D7.A, J24.1
- new net SEG10: D1S3.A, D2S8.A, D3S8.A, R17.2
- new net SEG11: D2S9.A, D3S9.A, DIS1.A, R18.2
- new net SEG12: D1S9.A, D2S11.A, D3S11.A, R21.2
- new net SEG13: D1S8.A, D2S10.A, D3S10.A, R20.2
- new net SEG14: D1S12.A, D2S14.A, D3S14.A, R22.2
- new net SEG8: D1S10.A, D2S12.A, D3S12.A, R16.2
- new net SEG9: D1S11.A, D2S13.A, D3S13.A, R19.2
- new net V_BATT1: C5.1, D4.A, D6.A, J13.2, R27.2, S6.2, U2.18, U2.4
- new net V_EXT: J9.1, S3.1
- new net V_EXT1: J21.1, S6.1
- net 7: now also R16.1, U2.26; no longer U1.13
- net GND: now also C3.2, R14.1
- net N$44: now also R1.1, R15.1; no longer R1.2
- net N$45: now also D1.C, R1.2; no longer D1.A, R1.1
- net N$46: now also D3.C, R15.2; no longer D1.C, J12.1
- net V_BATT: now also D2.A, S3.2; no longer J9.1, S3.1
Routing:
- net S$2: track 0.00 -> 137.2 mm
- net S$1: track 0.00 -> 137.2 mm
- net 18: track 0.00 -> 117.9 mm, vias 0 -> 2
- net 19: track 0.00 -> 109.6 mm, vias 0 -> 2
- net N$22: track 0.00 -> 93.8 mm, vias 1 -> 9
- net N$21: track 0.00 -> 74.0 mm, vias 1 -> 9
- net N$30: track 0.00 -> 67.6 mm
- net N$1: track 0.00 -> 67.6 mm, vias 0 -> 1
- net N$6: track 70.5 -> 3.00 mm, vias 1 -> 0
- net SEG12: track 0.00 -> 66.8 mm
- net V_BATT1: track 0.00 -> 63.0 mm, vias 0 -> 3
- net SEG11: track 0.00 -> 60.1 mm
- net SEG13: track 0.00 -> 60.1 mm
- net SEG14: track 0.00 -> 59.9 mm
- net SEG10: track 0.00 -> 56.7 mm
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- added copper zone on layer 1, net GND1
- added copper zone on layer 16, net GND1
- added copper zone on layer 16, net TAB1
- added copper zone on layer 1, net TAB2
- added copper zone on layer 16, net TAB5
- added copper zone on layer 1, net TAB6
- removed copper zone on layer 1, net MASKBTM
- removed copper zone on layer 16, net MASKTP
- removed copper zone on layer 16, net N$100
- removed copper zone on layer 16, net N$101
- removed copper zone on layer 16, net N$102
- removed copper zone on layer 16, net N$103
- removed copper zone on layer 16, net N$104
- removed copper zone on layer 16, net N$105
- removed copper zone on layer 1, net N$52
- removed copper zone on layer 1, net N$53
- removed copper zone on layer 1, net N$54
- removed copper zone on layer 1, net N$55
- removed copper zone on layer 1, net N$56
- removed copper zone on layer 1, net N$57
- removed copper zone on layer 1, net N$58
- removed copper zone on layer 1, net N$59
- removed copper zone on layer 1, net N$60
- removed copper zone on layer 16, net N$61
- removed copper zone on layer 16, net N$62
- removed copper zone on layer 16, net N$63
- removed copper zone on layer 16, net N$64
- removed copper zone on layer 16, net N$65
- removed copper zone on layer 16, net N$66
- removed copper zone on layer 16, net N$67
- removed copper zone on layer 16, net N$68
- removed copper zone on layer 16, net N$69
- removed copper zone on layer 1, net N$70
- removed copper zone on layer 1, net N$71
- removed copper zone on layer 1, net N$72
- removed copper zone on layer 1, net N$73
- removed copper zone on layer 1, net N$74
- removed copper zone on layer 1, net N$75
- removed copper zone on layer 1, net N$76
- removed copper zone on layer 1, net N$77
- removed copper zone on layer 1, net N$78
- removed copper zone on layer 16, net N$79
- removed copper zone on layer 16, net N$80
- removed copper zone on layer 16, net N$81
- removed copper zone on layer 16, net N$82
- removed copper zone on layer 16, net N$83
- removed copper zone on layer 16, net N$84
- removed copper zone on layer 16, net N$85
- removed copper zone on layer 16, net N$86
- removed copper zone on layer 16, net N$87
- removed copper zone on layer 1, net N$88
- removed copper zone on layer 1, net N$89
- removed copper zone on layer 1, net N$90
- removed copper zone on layer 1, net N$91
- removed copper zone on layer 1, net N$92
- removed copper zone on layer 1, net N$93
- removed copper zone on layer 1, net N$94
- removed copper zone on layer 1, net N$95
- removed copper zone on layer 1, net N$96
- removed copper zone on layer 16, net N$97
- removed copper zone on layer 16, net N$98
- removed copper zone on layer 16, net N$99
Other:
- board size 116.8 x 86.4 mm -> 116.8 x 77.2 mm
- board text added: "vscore"
