File: Hardware/Proto/0_8mm_Layers.sch (EAGLE design)
At the start: 59 parts, among them J1 AVR_SPI_PROG_3X2TESTPOINTS, Q1 220mA/50V/3.5Ω, Q2 220mA/50V/3.5Ω, Q3 220mA/50V/3.5Ω, U1 ATTINY861V-10MU

Commit message: v10
Parts:
- added C3: 0.1uF, SparkFun-Capacitors:0.1UF-0603-25V-(+80/-20%)
- added D2: IR PHOTOTRANS, SparkFun-LED:LED-IR0603
- added D3: IR LED, SparkFun-LED:LED-IR0603
- added R14, R15: 1k, SparkFun-Resistors:1KOHM-0603-1/10W-1%
Connections:
- net IR_DETECTOR renamed IR_DETECTOR_A
- removed net 7: U1.PA7(7/A6/AIN1/RX)
- removed net N$6: BT1.+, S3.P
- new net IR_DETECTOR_B: C3.1, D2.C, R14.2, U1.PA7(7/A6/AIN1/RX)
- new net N$1: BT1.+, S3.S
- new net N$51: D1.A, D3.A, J12.1
- new net V_EXT: J9.1, S3.O
- net GND: now also C3.2, R14.1
- net N$44: now also R1.1, R15.1; no longer R1.2
- net N$45: now also D1.C, R1.2; no longer D1.A, R1.1
- net N$46: now also D3.C, R15.2; no longer D1.C, J12.1
- net V_BATT: now also D2.A, S3.P; no longer J9.1, S3.O
Other:
- moved on the sheet: C1, D1, D23, J12, J2, R1, R12, S3
