File: hardware/BeanCounter_V10.sch (EAGLE design)
At the start: 58 parts, among them J1 AVR_SPI_PROG_3X2TESTPOINTS, Q1 220mA/50V/3.5Ω, Q2 220mA/50V/3.5Ω, Q3 220mA/50V/3.5Ω, U1 ATTINY861V-10MU

Commit message: Cleanup, add support files
Parts:
- removed D2, D23: IR PHOTOTRANS, SparkFun-LED:LED-IR0603
- added D1, D3: IR LED, SparkFun-LED:LED-IR0603
- added J12: (no value), SparkFun-Connectors:CONN_02
- added R1, R15: 1k, SparkFun-Resistors:1KOHM-0603-1/10W-1%
- added U$31, U$32: B19H1PT, IR:B19H1PT
Connections:
- new net N$31: D3.A, R15.2
- new net N$32: D1.A, R1.2
- new net N$44: J12.2, R1.1, R15.1
- new net N$51: D1.C, D3.C, J12.1
- net IR_DETECTOR_A: now also U$31.E1; no longer D23.C
- net IR_DETECTOR_B: now also U$32.E1; no longer D2.C
- net V_BATT: now also U$31.C1, U$32.C1; no longer D2.A, D23.A
Other:
- moved on the sheet: C1, R12
